Commit message: ur_macro

File: ur_description/urdf/inc/ur_macro.xacro (robot description, xacro)
@@ -316,4 +316,9 @@
       <child link="${prefix}tool0"/>
     </joint>
+    <group name="${prefix}arm_gripper">
+        <group name="${prefix}${name}_manipulator" />
+        <joint name="${prefix}gripper_grasp_point_joint"/>
+        <link name="${prefix}gripper_grasp_point"/>
+    </group>
   </xacro:macro>
 </robot>

Commit message: ur macro

File: ur_description/urdf/inc/ur_macro.xacro (robot description, xacro)
@@ -316,9 +316,19 @@
       <child link="${prefix}tool0"/>
     </joint>
-    <group name="${prefix}arm_gripper">
-        <group name="${prefix}${name}_manipulator" />
-        <joint name="${prefix}gripper_grasp_point_joint"/>
-        <link name="${prefix}gripper_grasp_point"/>
-    </group>
+    <!-- Virtual Grasp Point Link -->
+    <link name="${prefix}gripper_grasp_point">
+    </link>
+    <!-- Virtual Grasp Point Fixed Joint -->
+    <joint name="${prefix}gripper_grasp_point_joint" type="fixed">
+      <parent link="tool0"/>
+      <child link="${prefix}gripper_grasp_point"/>
+      <!-- Center between finger tips -->
+      <!-- Matching the table origin -->
+      <!--<origin rpy="1.570796325 0 -1.570796325" xyz="${0.213-0.024/2} 0 0"/>-->
+      <!-- Matching the convention -->
+      <!--z offset closed gripper from base to fingertip 162.8mm + force torque sensor 35mm-->
+      <origin rpy="0 0 0" xyz="0 0 0.1978"/>
+      <!--<limit effort="0" lower="0" upper="0" velocity="0"/>-->
+    </joint>
   </xacro:macro>
 </robot>

Commit message: use correct ft sensor length

File: ur_description/urdf/inc/ur_macro.xacro (robot description, xacro)
@@ -328,5 +328,5 @@
       <!-- Matching the convention -->
       <!--z offset closed gripper from base to fingertip 162.8mm + force torque sensor 35mm-->
-      <origin rpy="0 0 0" xyz="0 0 0.1978"/>
+      <origin rpy="0 0 0" xyz="0 0 0.035"/>
       <!--<limit effort="0" lower="0" upper="0" velocity="0"/>-->
     </joint>
